File: hardware/medidor-energia.kicad_sch (KiCad schematic)
At the start: 54 parts, among them J1 Bornera 5 V, J2 Jack 3,5 mm de panel (pinza S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, J3 Jack 3,5 mm de panel (pinza S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, J4 Bornera red L/N, J5 Bornera ZMPT, J6 LCD (VCC GND DIN CS DC BL CLK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, J7 Reserva ADC1, SW1 Pulsador de panel 12 mm NA, SW2 Pulsador de panel 12 mm NA, U1 ESP32-DevKitC V4 (38 pines), U2 Módulo ZMPT101B

Commit message: Correcciones de la revisión del diseño
- Firmware: la adquisición la despierta un temporizador de hardware (antes esperaba de forma activa
  y bloqueaba el arranque); eventos de Wi-Fi en el núcleo 0; tarea de adquisición creada al final.
- Fase: historia de tensión de 8 muestras, corrección de −8° a +11° con fase del ZMPT101B y de cada
  pinza; calibración guardada en NVS desde la consola serie (comando cal).
- Ventanas por cantidad de muestras cuando no hay cruces por cero (ZMPT101B desconectado).
- Hardware: C5 y C6 vuelven a VBIAS (antes a GND, acoplaban los canales ~1 %); PCB re-ruteada con
  2 puentes; placa perforada y simulación actualizadas.
- README: aislamiento del ZMPT101B y criterio de 100 MΩ, alimentación por USB, tierra, prueba de
  cortocircuito, calibración de fase y nuevas pruebas del cálculo.
Parts:
- removed C10, C11: 100n, Capacitor_THT:C_Disc_D5.0mm_W2.5mm_P5.00mm, symbol Device:C
- removed C7: 10u 16V, Capacitor_THT:CP_Radial_D5.0mm_P2.50mm, symbol Device:C_Polarized
- removed D5, D6, D7: BAT85, Diode_THT:D_DO-35_SOD27_P7.62mm_Horizontal, symbol Device:D_Schottky
- removed R11: 330, Resistor_THT:R_Axial_DIN0207_L6.3mm_D2.5mm_P10.16mm_Horizontal, symbol Device:R
- removed TP7: V_ADC, TestPoint:TestPoint_Loop_D2.50mm_Drill1.0mm, symbol Connector:TestPoint
- removed TP9: GND, TestPoint:TestPoint_Loop_D2.50mm_Drill1.0mm, symbol Connector:TestPoint
- removed U2: Módulo ZMPT101B, symbol Medidor:ZMPT101B_Modulo
- added D10: LED verde 3 mm, LED_THT:LED_D3.0mm, symbol Device:LED
- added D8: LED verde 5 mm (panel), Connector_PinHeader_2.54mm:PinHeader_1x02_P2.54mm_Vertical, symbol Device:LED
- added J3: Jack 3,5 mm de panel (pinza SCT-013-000 CH2), Medidor:Cable_Jack_Panel, symbol Connector_Audio:AudioJack3
- added J4: Bornera red L/N, TerminalBlock_Phoenix:TerminalBlock_Phoenix_MKDS-1,5-2-5.08_1x02_P5.08mm_Horizontal, symbol Connector:Screw_Terminal_01x02
- added R13: 10k, Resistor_THT:R_Axial_DIN0207_L6.3mm_D2.5mm_P10.16mm_Horizontal, symbol Device:R
- added R4: 10k 1%, Resistor_THT:R_Axial_DIN0207_L6.3mm_D2.5mm_P10.16mm_Horizontal, symbol Device:R
- added R7: 11k 1%, Resistor_THT:R_Axial_DIN0207_L6.3mm_D2.5mm_P10.16mm_Horizontal, symbol Device:R
- added R8: 13k 1%, Resistor_THT:R_Axial_DIN0207_L6.3mm_D2.5mm_P10.16mm_Horizontal, symbol Device:R
- added TP1: +5V, TestPoint:TestPoint_Loop_D2.50mm_Drill1.0mm, symbol Connector:TestPoint
- added TP4: CH1_ADC, TestPoint:TestPoint_Loop_D2.50mm_Drill1.0mm, symbol Connector:TestPoint
- C10: renamed from R12; value 10k -> 100n; footprint Resistor_THT:R_Axial_DIN0207_L6.3mm_D2.5mm_P10.16mm_Horizontal -> Capacitor_THT:C_Disc_D5.0mm_W2.5mm_P5.00mm; symbol Device:R -> Device:C
- C11: renamed from R13; value 10k -> 100n; footprint Resistor_THT:R_Axial_DIN0207_L6.3mm_D2.5mm_P10.16mm_Horizontal -> Capacitor_THT:C_Disc_D5.0mm_W2.5mm_P5.00mm; symbol Device:R -> Device:C
- C6: renamed from R6; value 3,3k 1% -> 47n C0G; footprint Resistor_THT:R_Axial_DIN0207_L6.3mm_D2.5mm_P10.16mm_Horizontal -> Capacitor_THT:C_Disc_D5.0mm_W2.5mm_P5.00mm; symbol Device:R -> Device:C
- C7: renamed from R4; value 10k 1% -> 10u 16V; footprint Resistor_THT:R_Axial_DIN0207_L6.3mm_D2.5mm_P10.16mm_Horizontal -> Capacitor_THT:CP_Radial_D5.0mm_P2.50mm; symbol Device:R -> Device:C_Polarized
- C9: renamed from R7; value 11k 1% -> 27n C0G; footprint Resistor_THT:R_Axial_DIN0207_L6.3mm_D2.5mm_P10.16mm_Horizontal -> Capacitor_THT:C_Disc_D7.5mm_W5.0mm_P5.00mm; symbol Device:R -> Device:C
- D4: renamed from C6; value 47n C0G -> BAT85; footprint Capacitor_THT:C_Disc_D5.0mm_W2.5mm_P5.00mm -> Diode_THT:D_DO-35_SOD27_P7.62mm_Horizontal; symbol Device:C -> Device:D_Schottky
- D6: renamed from R8; value 13k 1% -> BAT85; footprint Resistor_THT:R_Axial_DIN0207_L6.3mm_D2.5mm_P10.16mm_Horizontal -> Diode_THT:D_DO-35_SOD27_P7.62mm_Horizontal; symbol Device:R -> Device:D_Schottky
- D7: renamed from C9; value 27n C0G -> BAT85; footprint Capacitor_THT:C_Disc_D7.5mm_W5.0mm_P5.00mm -> Diode_THT:D_DO-35_SOD27_P7.62mm_Horizontal; symbol Device:C -> Device:D_Schottky
- R11: renamed from D10; value LED verde 3 mm -> 330; footprint LED_THT:LED_D3.0mm -> Resistor_THT:R_Axial_DIN0207_L6.3mm_D2.5mm_P10.16mm_Horizontal; symbol Device:LED -> Device:R
- R12: renamed from D8; value LED verde 5 mm (panel) -> 10k; footprint Connector_PinHeader_2.54mm:PinHeader_1x02_P2.54mm_Vertical -> Resistor_THT:R_Axial_DIN0207_L6.3mm_D2.5mm_P10.16mm_Horizontal; symbol Device:LED -> Device:R
- R2: renamed from J3; value Jack 3,5 mm de panel (pinza SCT-013-000 CH2) -> 47 1% 1/4 W (burden); footprint Medidor:Cable_Jack_Panel -> (none); symbol Connector_Audio:AudioJack3 -> Device:R
- R6: renamed from R2; value 47 1% 1/4 W (burden) -> 3,3k 1%; footprint (none) -> Resistor_THT:R_Axial_DIN0207_L6.3mm_D2.5mm_P10.16mm_Horizontal
- TP2: renamed from TP1; value +5V -> +3V3
- TP3: renamed from TP2; value +3V3 -> VBIAS
- TP5: renamed from TP3; value VBIAS -> CH2_ADC
- TP6: renamed from TP4; value CH1_ADC -> ZMPT_OUT
- TP7: renamed from TP5; value CH2_ADC -> V_ADC
- TP8: renamed from TP6; value ZMPT_OUT -> GND
- U2: renamed from J4; value Bornera red L/N -> Módulo ZMPT101B; footprint TerminalBlock_Phoenix:TerminalBlock_Phoenix_MKDS-1,5-2-5.08_1x02_P5.08mm_Horizontal -> (none); symbol Connector:Screw_Terminal_01x02 -> Medidor:ZMPT101B_Modulo
- renumbered D4 to D5, TP8 to TP9
Connections:
- net +3V3: now also D4.1 (K), D6.1 (K), R12.1, TP2.1, R13.1; no longer C10.1, C11.1, D5.1 (K), TP3.1
- net +5V: now also U2.3 (VCC), TP1.1; no longer TP2.1
- net CH1_ADC: now also TP4.1; no longer TP6.1
- net CH2_ADC: now also C6.1, D4.2 (A), D5.1 (K), R6.2, TP5.1; no longer C6.2, D4.1, D5.2 (A), TP7.1
- net GND: now also C10.2, C11.2, C9.2, D5.2 (A), TP8.1, U2.5 (GND), D10.1 (K), D8.1 (K), R4.2, R8.2; no longer C5.2, D4.2, D6.2, R11.1 (K), R12.1 (K)
- net LED_EST: now also R11.1
- net SW1: now also C10.1, R12.2; no longer C10.2
- net SW2: now also C11.1, R13.2; no longer C11.2
- net VBIAS: now also C5.2, C6.2, R2.1, TP3.1, J3.S, R4.1; no longer R2.S, R6.1, TP5.1
- net V_ADC: now also C9.1, D6.2 (A), TP7.1, R7.2, R8.1; no longer C9.2, D6.1
- net ZMPT_OUT: now also TP6.1, U2.4 (OUT), R7.1; no longer C9.1, TP8.1
- net at R11.2: now also D8.2 (A); no longer R15.2
- net at F1.1: now also J4.1 (Pin_1); no longer U2.1 (Pin_1)
- net at U2.2 (N): now also J4.2 (Pin_2)
- net at F1.2: now also U2.1 (L)
- new net: J3.T, R2.2, R6.1
- new net: D10.2 (A), R15.2
Other:
- note added: "La corriente de la pinza y la del filtro (C5, C6) cierran en VBIAS; al divisor solo llega la corriente de entrada del ADC: un divisor sirve a los dos canales."
- note removed: "La corriente de la pinza circula solo por el burden; VBIAS solo ve la corriente de entrada del ADC, por eso un divisor sirve a los dos canales."
- moved on the sheet: D5, R6, TP2, TP3, TP5, TP6, TP7, TP8, TP9
